Commit message: Nagemeten chassismaten en lidarpositie, udev-regel voor de lidar
Co-Authored-By: Claude Opus 5.5 <noreply@anthropic.com>

File: src/wave_rover_description/urdf/wave_rover.urdf.xacro (robot description, xacro)
@@ -1,13 +1,12 @@
 <?xml version="1.0"?>
-<!-- Wave Rover. Chassismaten zijn een schatting: nameten en aanpassen.
-     Posities van lidar, camera en IMU komen uit de legacy-opstelling. -->
+<!-- Wave Rover. Maten nagemeten op 2026-10-21; positie van camera en IMU nog geschat. -->
 <robot name="wave_rover" xmlns:xacro="http://www.ros.org/wiki/xacro">
-  <xacro:property name="body_length" value="0.23"/>
-  <xacro:property name="body_width" value="0.16"/>
+  <xacro:property name="body_length" value="0.18"/>
+  <xacro:property name="body_width" value="0.17"/>
   <xacro:property name="body_height" value="0.06"/>
   <xacro:property name="wheel_radius" value="0.04"/>
   <xacro:property name="wheel_width" value="0.035"/>
-  <xacro:property name="wheel_base" value="0.12"/>
-  <xacro:property name="track_width" value="0.17"/>
+  <xacro:property name="wheel_base" value="0.10"/>
+  <xacro:property name="track_width" value="0.12"/>
   <material name="body"><color rgba="0.15 0.15 0.15 1"/></material>
   <material name="wheel"><color rgba="0.05 0.05 0.05 1"/></material>
@@ -53,5 +52,6 @@
     <origin xyz="0 0 0.01"/>
   </joint>
-  <!-- RPLidar C1; frame-naam "laser" is de standaard van rplidar_ros. -->
+  <!-- RPLidar C1; frame-naam "laser" is de standaard van rplidar_ros.
+       Op 70% van de lengte richting achterkant; laser op 20 cm boven de grond. -->
   <link name="laser">
     <visual>
@@ -63,5 +63,5 @@
     <parent link="base_link"/>
     <child link="laser"/>
-    <origin xyz="0.1 0 0.16"/>
+    <origin xyz="${body_length/2 - 0.7*body_length} 0 ${0.20 - wheel_radius}"/>
   </joint>
   <link name="camera_link">

Commit message: Module-manager: modules op vraag starten en stoppen
- wave_rover_manager: /modules/<naam>/enable (SetBool) en /modules/status (JSON)
- config/modules.yaml met de lidar als eerste module
- Lidar 180 graden gedraaid in de URDF, RViz gebruikt rviz_imu_plugin

Co-Authored-By: Claude Opus 5.5 <noreply@anthropic.com>

File: src/wave_rover_description/urdf/wave_rover.urdf.xacro (robot description, xacro)
@@ -53,5 +53,6 @@
   </joint>
   <!-- RPLidar C1; frame-naam "laser" is de standaard van rplidar_ros.
-       Op 70% van de lengte richting achterkant; laser op 20 cm boven de grond. -->
+       Op 70% van de lengte richting achterkant; laser op 20 cm boven de grond.
+       De lidar is gemonteerd met zijn pijl naar achteren: 180 graden gedraaid. -->
   <link name="laser">
     <visual>
@@ -63,5 +64,5 @@
     <parent link="base_link"/>
     <child link="laser"/>
-    <origin xyz="${body_length/2 - 0.7*body_length} 0 ${0.20 - wheel_radius}"/>
+    <origin xyz="${body_length/2 - 0.7*body_length} 0 ${0.20 - wheel_radius}" rpy="0 0 ${pi}"/>
   </joint>
   <link name="camera_link">

Commit message: Odometrie- en SLAM-modules, camera in URDF, opstartoverzicht
- odometry: rf2o_laser_odometry + robot_localization (EKF met IMU-gyro)
- slam: slam_toolbox (online async), RViz-config mapping.rviz
- rf2o, robot_localization en slam_toolbox in het Docker-image
- Camera plat op het chassis in de URDF
- scripts/boot_history.sh: toont abrupt geëindigde sessies (bevriezing/watchdog)

Co-Authored-By: Claude Opus 5.5 <noreply@anthropic.com>

File: src/wave_rover_description/urdf/wave_rover.urdf.xacro (robot description, xacro)
@@ -1,4 +1,4 @@
 <?xml version="1.0"?>
-<!-- Wave Rover. Maten nagemeten op 2026-10-21; positie van camera en IMU nog geschat. -->
+<!-- Wave Rover. Maten nagemeten op 2026-10-21; positie van de IMU nog geschat. -->
 <robot name="wave_rover" xmlns:xacro="http://www.ros.org/wiki/xacro">
   <xacro:property name="body_length" value="0.18"/>
@@ -72,8 +72,9 @@
     </visual>
   </link>
+  <!-- Camera ligt plat op het chassis, in het midden, 4 cm van de voorrand. -->
   <joint name="camera_joint" type="fixed">
     <parent link="base_link"/>
     <child link="camera_link"/>
-    <origin xyz="0.12 0 0.26" rpy="0 0.1745 0"/>
+    <origin xyz="${body_length/2 - 0.04} 0 ${body_height/2 + 0.015}"/>
   </joint>
 </robot>

Commit message: SLAM via officiële lifecycle-launch, drifttest, lidar 3 cm naar links
Co-Authored-By: Claude Opus 5.5 <noreply@anthropic.com>

File: src/wave_rover_description/urdf/wave_rover.urdf.xacro (robot description, xacro)
@@ -53,5 +53,5 @@
   </joint>
   <!-- RPLidar C1; frame-naam "laser" is de standaard van rplidar_ros.
-       Op 70% van de lengte richting achterkant; laser op 20 cm boven de grond.
+       Op 70% van de lengte richting achterkant, 3 cm links van het midden; laser op 20 cm boven de grond.
        De lidar is gemonteerd met zijn pijl naar achteren: 180 graden gedraaid. -->
   <link name="laser">
@@ -64,5 +64,5 @@
     <parent link="base_link"/>
     <child link="laser"/>
-    <origin xyz="${body_length/2 - 0.7*body_length} 0 ${0.20 - wheel_radius}" rpy="0 0 ${pi}"/>
+    <origin xyz="${body_length/2 - 0.7*body_length} 0.03 ${0.20 - wheel_radius}" rpy="0 0 ${pi}"/>
   </joint>
   <link name="camera_link">

Commit message: Fase 4: lage obstakels met de camera (module floor_obstacles -> /floor_scan, Nav2 floor_layer)
- Depth Anything V2 Small (TensorRT, ingang ruwe RGB-bytes) + vaste camerageometrie:
  vloer per beeld robuust gepast, alles wat eruit steekt = obstakel op het contactpunt
- Nav2: eigen ObstacleLayer in local en global costmap; geen wissen in de blinde zone,
  obstacle_max_range onder range_max zodat inf enkel wist
- kalibratie (scripts/calibrate_floor.py): lens 10,5 cm, f 989,5 px, pitch -0,011 rad;
  URDF-camerahoogte aangepast
- scripts/export_depth.py

Co-Authored-By: Claude Opus 5.5 <noreply@anthropic.com>

File: src/wave_rover_description/urdf/wave_rover.urdf.xacro (robot description, xacro)
@@ -72,9 +72,10 @@
     </visual>
   </link>
-  <!-- Camera ligt plat op het chassis, in het midden, 4 cm van de voorrand. -->
+  <!-- Camera ligt plat op het chassis, in het midden, 4 cm van de voorrand; midden van de
+       lens 10,5 cm boven de vloer (gemeten 28-10-2026). -->
   <joint name="camera_joint" type="fixed">
     <parent link="base_link"/>
     <child link="camera_link"/>
-    <origin xyz="${body_length/2 - 0.04} 0 ${body_height/2 + 0.015}"/>
+    <origin xyz="${body_length/2 - 0.04} 0 ${0.105 - wheel_radius}"/>
   </joint>
 </robot>
